File: pcb/gullwing/gullwing.kicad_pcb (KiCad board)
At the start: 2 copper layers, 108 parts, among them J1 XF2M-1415-1A, J2 XF2M-1415-1A, J3 XF2M-1415-1A, J4 XF2M-1415-1A, U1 RP2040_Zero

Commit message: done -- first pass
Parts:
- removed ? (x2): , 
- added 3.3v1: TestPoint, TestPoint:TestPoint_Pad_1.0x1.0mm, F.Cu at (228.6, 134.7)
- added DR1: TestPoint, TestPoint:TestPoint_Pad_1.0x1.0mm, F.Cu at (224.6, 134.7)
- added PAD8: , MountingHole_2.2mm_M2, F.Cu at (190.2, 145.0)
- added PAD8: , MountingHole_2.2mm_M2, F.Cu at (245.9, 145.0)
- added PAD8: , MountingHole_2.2mm_M2, F.Cu at (224.8, 105.8)
- added PAD8: , MountingHole_2.2mm_M2, F.Cu at (170.3, 78.8)
- added PAD8: , MountingHole_2.2mm_M2, F.Cu at (209.2, 168.3)
- added PAD8: , MountingHole_2.2mm_M2, F.Cu at (225.3, 168.3)
- added PAD8: , MountingHole_2.2mm_M2, F.Cu at (211.4, 105.8)
- added PAD8: , MountingHole_2.2mm_M2, F.Cu at (266.8, 78.5)
- added RSTb1: TestPoint, TestPoint:TestPoint_Pad_1.0x1.0mm, F.Cu at (226.6, 134.7)
- added SCL1: TestPoint, TestPoint:TestPoint_Pad_1.0x1.0mm, F.Cu at (232.6, 134.7)
- added SDA1: TestPoint, TestPoint:TestPoint_Pad_1.0x1.0mm, F.Cu at (234.6, 134.7)
- added gnd1: TestPoint, TestPoint:TestPoint_Pad_1.0x1.0mm, F.Cu at (230.6, 134.7)
- added mb2: Mouse_Bites_5, ScottoKeebs_Miscellaneous:Mouse_Bites_5, F.Cu at (212.9, 97.5)
- added mb2: Mouse_Bites_5, ScottoKeebs_Miscellaneous:Mouse_Bites_5, F.Cu at (218.1, 102.0)
- added mb2: Mouse_Bites_5, ScottoKeebs_Miscellaneous:Mouse_Bites_5, F.Cu at (223.3, 97.5)
- added mb2: Mouse_Bites_5, ScottoKeebs_Miscellaneous:Mouse_Bites_5, F.Cu at (218.1, 172.2)
- moved D39 9.20 mm to (312.2, 153.6)
- moved D40 9.20 mm to (330.2, 153.6)
- moved PAD8 9.20 mm to (321.2, 138.8)
- moved SW39 9.20 mm to (312.2, 149.0)
- moved SW40 9.20 mm to (330.2, 149.0)
- moved D20 8.70 mm to (329.8, 126.0)
- moved D21 8.70 mm to (301.2, 89.4)
- moved D23 8.70 mm to (310.6, 122.1)
- moved D26 8.70 mm to (291.7, 122.4)
- moved D30 8.70 mm to (267.6, 156.4)
- moved PAD6 8.70 mm to (311.9, 90.2)
- moved SW19 8.70 mm to (326.4, 104.5)
- moved SW28 8.70 mm to (268.5, 111.4)
- moved SW29 8.70 mm to (274.3, 127.3)
- moved D12 8.70 mm to (125.6, 122.1)
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Connections:
- J3 pad 10: unconnected-(J3-Pad10) -> GND
- J3 pad 11: unconnected-(J3-Pad11) -> +3V3
- J4 pad 4: unconnected-(J4-Pad4) -> +3V3
- J4 pad 5: unconnected-(J4-Pad5) -> GND
- U1 pad 10: unconnected-(U1-9-Pad10) -> scl
- U1 pad 8: unconnected-(U1-7-Pad8) -> dr
- U1 pad 9: unconnected-(U1-8-Pad9) -> sda
Routing:
- net +3V3: track 0.00 -> 122.8 mm, vias 0 -> 3
- net GND: track 0.00 -> 119.7 mm, vias 0 -> 3
- net scl: track 13.3 -> 113.0 mm, vias 3 -> 4
- net dr: track 12.1 -> 108.1 mm
- net sda: track 12.3 -> 107.9 mm, vias 3 -> 4
- net r0: track 73.6 -> 93.4 mm, vias 1 -> 3
- net r1: track 74.2 -> 93.1 mm, vias 1 -> 3
- net r3: track 75.4 -> 94.1 mm
- net r2: track 74.6 -> 93.3 mm
- net c9: track 143.6 -> 155.9 mm
- net c4: track 151.3 -> 163.2 mm
- net c3: track 130.5 -> 142.4 mm
- net c0: track 169.7 -> 180.0 mm
- net c8: track 122.2 -> 132.2 mm
- net c5: track 175.4 -> 185.4 mm
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Other:
- board outline added: 244.6 x 107.8 mm
- board text removed: "TODO: ROUTE SDA/SCL/DR TO MCU PINS + TOUCH PAD"

Commit message: done -- ready for export
Parts:
- removed the PAD8 at (190.2, 145.0)
- removed the PAD8 at (245.9, 145.0)
- added G***: LOGO, images_lib:smiley, F.Cu at (139.0, 153.8)
- added G***: LOGO, images_lib:smiley, F.Cu at (297.5, 153.8)
- added J5: XF2M-0615-1A, Connector_FFC-FPC:XF2M06151A, B.Cu at (232.0, 147.0)
- added PAD8: , MountingHole_2.2mm_M2, F.Cu at (200.1, 86.7)
- added PAD8: , MountingHole_2.2mm_M2, F.Cu at (236.1, 86.7)
- moved PAD8 12.7 mm to (236.2, 111.4)
- moved PAD8 12.7 mm to (200.1, 111.4)
- moved 3.3v1 5.00 mm to (228.6, 129.7)
- moved DR1 5.00 mm to (224.6, 129.7)
- moved RSTb1 5.00 mm to (226.6, 129.7)
- moved SCL1 5.00 mm to (232.6, 129.7)
- moved SDA1 5.00 mm to (234.6, 129.7)
- moved gnd1 5.00 mm to (230.6, 129.7)
- moved J1 2.00 mm to (182.8, 75.0), turned to 90 degrees
- moved PAD8 1.65 mm to (210.9, 168.3)
- moved J2 1.50 mm to (203.2, 75.0), turned to -90 degrees
- moved J4 1.50 mm to (233.1, 75.0), turned to 90 degrees
- turned J3 to -90 degrees
Connections:
- J1 pad 1: r0l -> c0
- J1 pad 10: c4 -> unconnected-(J1-Pad10)
- J1 pad 11: c3 -> r3l
- J1 pad 12: c2 -> r2l
- J1 pad 13: c1 -> r1l
- J1 pad 14: c0 -> r0l
- J1 pad 2: r1l -> c1
- J1 pad 3: r2l -> c2
- J1 pad 4: r3l -> c3
- J1 pad 5: unconnected-(J1-Pad5) -> c4
- J2 pad 1: c0 -> r0
- J2 pad 10: unconnected-(J2-Pad10) -> c4
- J2 pad 11: r3 -> c3
- J2 pad 12: r2 -> c2
- J2 pad 13: r1 -> c1
- J2 pad 14: r0 -> c0
- J2 pad 2: c1 -> r1
- J2 pad 3: c2 -> r2
- J2 pad 4: c3 -> r3
- J2 pad 5: c4 -> unconnected-(J2-Pad5)
- J3 pad 1: c5 -> scl
- J3 pad 10: GND -> c9
- J3 pad 11: +3V3 -> c8
- J3 pad 12: dr -> c7
- J3 pad 13: sda -> c6
- J3 pad 14: scl -> c5
- J3 pad 2: c6 -> sda
- J3 pad 3: c7 -> dr
- J3 pad 4: c8 -> +3V3
- J3 pad 5: c9 -> GND
- J3 pad 6: r3r -> r0r
- J3 pad 7: r2r -> r1r
- J3 pad 8: r1r -> r2r
- J3 pad 9: r0r -> r3r
- J4 pad 1: scl -> c5
- J4 pad 10: c9 -> GND
- J4 pad 11: c8 -> +3V3
- J4 pad 12: c7 -> dr
- J4 pad 13: c6 -> sda
- J4 pad 14: c5 -> scl
- J4 pad 2: sda -> c6
- J4 pad 3: dr -> c7
- J4 pad 4: +3V3 -> c8
- J4 pad 5: GND -> c9
- J4 pad 6: r0 -> r3
- J4 pad 7: r1 -> r2
- J4 pad 8: r2 -> r1
- J4 pad 9: r3 -> r0
Routing:
- net +3V3: track 122.8 -> 176.7 mm, vias 3 -> 5
- net dr: track 108.1 -> 132.3 mm
- net sda: track 107.9 -> 130.4 mm
- net scl: track 113.0 -> 132.8 mm
- net GND: track 119.7 -> 105.6 mm, vias 3 -> 20
- net r1l: track 225.0 -> 237.8 mm
- net r2l: track 233.8 -> 246.4 mm
- net r3l: track 260.2 -> 271.6 mm
- net r0l: track 201.3 -> 212.6 mm
- net r3r: track 258.7 -> 264.6 mm
- net r1r: track 204.5 -> 210.1 mm
- net r0r: track 189.6 -> 194.9 mm
- net r3: track 94.1 -> 98.3 mm
- net r2: track 93.3 -> 96.9 mm
- net r0: track 93.4 -> 96.6 mm, vias 3 -> 1
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- added copper zone on B.Cu, net GND
- added copper zone on F.Cu, net GND
Other:
- outline, holes or cut-outs redrawn
- board text added: "gullwing v1.0"
