File: pcb/gullwing/gullwing.kicad_sch (KiCad schematic)
At the start: 93 parts, among them J1 XF2M-1415-1A, J2 XF2M-1415-1A, J3 XF2M-1415-1A, J4 XF2M-1415-1A, U1 RP2040_Zero

Commit message: done -- first pass
Parts:
- added 3.3v1, DR1, RSTb1, SCL1, SDA1, gnd1: TestPoint, TestPoint:TestPoint_Pad_1.0x1.0mm, symbol Connector:TestPoint
Connections:
- net +3V3: now also J3.11, J4.4, 3.3v1.1, RSTb1.1
- net GND: now also J3.10, J4.5, gnd1.1
- net dr: now also U1.8 (7), DR1.1
- net scl: now also U1.10 (9), SCL1.1
- net sda: now also U1.9 (8), SDA1.1

Commit message: done -- ready for export
Parts:
- added J5: XF2M-0615-1A, Connector_FFC-FPC:XF2M06151A, symbol XF2M-0615-1A:XF2M-0615-1A
- SW1, SW10, SW11, SW12, SW13, SW14, SW15, SW16, SW17, SW18, SW19, SW2, SW20, SW21, SW22, SW23, SW24, SW25, SW26, SW27, SW28, SW29, SW3, SW30, SW31, SW32, SW33, SW34, SW35, SW36, SW37, SW38, SW39, SW4, SW40, SW5, SW6, SW7, SW8, SW9, U1: now not fitted
Connections:
- net +3V3: now also J3.4, J4.11, J5.2, J5.4; no longer J3.11, J4.4
- net GND: now also J3.5, J4.10, J5.3; no longer J3.10, J4.5
- net c0: now also J1.1, J2.14; no longer J1.14, J2.1
- net c1: now also J1.2, J2.13; no longer J1.13, J2.2
- net c2: now also J1.3, J2.12; no longer J1.12, J2.3
- net c3: now also J1.4, J2.11; no longer J1.11, J2.4
- net c4: now also J1.5, J2.10; no longer J1.10, J2.5
- net c5: now also J3.14, J4.1; no longer J3.1, J4.14
- net c6: now also J3.13, J4.2; no longer J3.2, J4.13
- net c7: now also J3.12, J4.3; no longer J3.3, J4.12
- net c8: now also J3.11, J4.4; no longer J3.4, J4.11
- net c9: now also J3.10, J4.5; no longer J3.5, J4.10
- net dr: now also J3.3, J4.12, J5.1; no longer J3.12, J4.3
- net r0: now also J2.1, J4.9; no longer J2.14, J4.6
- net r0l: now also J1.14; no longer J1.1
- net r0r: now also J3.6; no longer J3.9
- net r1: now also J2.2, J4.8; no longer J2.13, J4.7
- net r1l: now also J1.13; no longer J1.2
- net r1r: now also J3.7; no longer J3.8
- net r2: now also J2.3, J4.7; no longer J2.12, J4.8
- net r2l: now also J1.12; no longer J1.3
- net r2r: now also J3.8; no longer J3.7
- net r3: now also J2.4, J4.6; no longer J2.11, J4.9
- net r3l: now also J1.11; no longer J1.4
- net r3r: now also J3.9; no longer J3.6
- net scl: now also J3.1, J4.14, J5.5; no longer J3.14, J4.1
- net sda: now also J3.2, J4.13, J5.6; no longer J3.13, J4.2
- no-connect marks 0 -> 23
Other:
- moved on the sheet: 3.3v1, DR1, RSTb1, SCL1, SDA1, gnd1
